Commit message: Replace rotors dae with fuel

File: urdf/iris/iris_depthcam.xacro (robot description, xacro)
@@ -7,5 +7,5 @@
     name="camera" parent_link="${namespace}/base_link"
     update_rate="10" min_range="0.05" max_range="8.0" field_of_view="1.347198">
-    <origin xyz="0.03 0 -0.06" rpy="0 0 0" />
+    <origin xyz="0.03 0 -0.075" rpy="0 0 0" />
   </xacro:depth_camera>
   <!-- ray sensors -->
@@ -18,8 +18,8 @@
     offY_left="0.06"
     offY_right="-0.06"
-    offZ_up="0.055"
+    offZ_up="0.07"
     offZ_horizon1="-0.01"
     offZ_horizon2="0.01"
-    offZ_down="-0.085"
+    offZ_down="-0.1"
   />
 </robot>

File: urdf/parts/rotors_custom/iris.xacro (robot description, xacro)
@@ -5,5 +5,5 @@
   <xacro:property name="rotor_velocity_slowdown_sim" value="10" />
   <xacro:property name="use_mesh_file" value="true" />
-  <xacro:property name="mesh_file" value="package://rotors_description/meshes/iris.dae" />
+  <xacro:property name="mesh_file" value="https://fuel.ignitionrobotics.org/1.0/OpenRobotics/models/X3 UAV/4/files/meshes/x3.dae" />
   <xacro:property name="mass" value="1.5" /> <!-- [kg] -->
   <xacro:property name="body_width" value="0.47" /> <!-- [m] -->

File: urdf/parts/rotors_custom/multirotor_base.xacro (robot description, xacro)
@@ -102,5 +102,5 @@
           </xacro:if>
           <xacro:unless value="${use_own_mesh}">
-            <mesh filename="package://rotors_description/meshes/propeller_${direction}.dae"
+            <mesh filename="https://fuel.ignitionrobotics.org/1.0/OpenRobotics/models/X3 UAV/4/files/meshes/propeller_cw.dae"
               scale="${radius_rotor} ${radius_rotor} ${radius_rotor}" /> <!-- The propeller meshes have a radius of 1m -->
             <!-- <box size="${2*radius_rotor} 0.01 0.005"/> -->
