Commit message: Replace range plugin (temporary)

File: urdf/parts/range/range1ray.urdf.xacro (robot description, xacro)
@@ -5,5 +5,5 @@
 -->
 <robot xmlns:xacro="http://ros.org/wiki/xacro">
-  <xacro:macro name="sonar_sensor" params="name parent *origin ros_topic update_rate min_range max_range field_of_view ray_count">
+  <xacro:macro name="sonar_sensor" params="name parent *origin topic update_rate min_range max_range field_of_view ray_count">
     <joint name="${name}_joint" type="fixed">
       <xacro:insert_block name="origin" />
@@ -31,6 +31,8 @@
     </link>
     <gazebo reference="${namespace}/${name}_link">
-      <sensor type="ray" name="${name}">
-        <pose>0 0 0 0 0 0</pose>
+      <!-- since ray sensor is not implemented in Ignition Gazebo yet, gpu_lidar is used instead -->
+      <sensor type="gpu_lidar" name="${name}">
+        <pose relative_to='${namespace}/${name}_link'>0 0 0 0 0 0</pose>
+        <topic>${namespace}/${topic}</topic>
         <visualize>true</visualize>
         <update_rate>${update_rate}</update_rate>
@@ -56,4 +58,5 @@
           </range>
         </ray>
+        <!--
         <plugin filename="libgazebo_ros_range.so" name="gazebo_ros_range">
           <gaussianNoise>0.005</gaussianNoise>
@@ -65,4 +68,5 @@
           <fov>${field_of_view}</fov>
         </plugin>
+        -->
       </sensor>
     </gazebo>

File: urdf/parts/range/range1ray_14align.urdf.xacro (robot description, xacro)
@@ -6,57 +6,57 @@
       <xacro:include filename="$(find ign_gazebo_prac)/urdf/parts/range/range1ray.urdf.xacro" />
       <!-- front -->
-      <xacro:sonar_sensor name="ray_front" parent="${parent_link}" ros_topic="range_front" update_rate="${rate}" min_range="${min}" max_range="${max}" field_of_view="${ray_fov*M_PI/180}" ray_count="1">
+      <xacro:sonar_sensor name="ray_front" parent="${parent_link}" topic="range_front" update_rate="${rate}" min_range="${min}" max_range="${max}" field_of_view="${ray_fov*M_PI/180}" ray_count="1">
         <origin xyz="${offX_front} 0.0 ${offZ_horizon1}" rpy="0 0 0" />
       </xacro:sonar_sensor>
       <!-- right front -->
-      <xacro:sonar_sensor name="ray_rfront" parent="${parent_link}" ros_topic="range_rfront" update_rate="${rate}" min_range="${min}" max_range="${max}" field_of_view="${ray_fov*M_PI/180}" ray_count="1">
+      <xacro:sonar_sensor name="ray_rfront" parent="${parent_link}" topic="range_rfront" update_rate="${rate}" min_range="${min}" max_range="${max}" field_of_view="${ray_fov*M_PI/180}" ray_count="1">
         <origin xyz="${offX_front} ${offY_right} ${offZ_horizon1}" rpy="0 0 ${-45*M_PI/180}" />
       </xacro:sonar_sensor>
       <!-- left front -->
-      <xacro:sonar_sensor name="ray_lfront" parent="${parent_link}" ros_topic="range_lfront" update_rate="${rate}" min_range="${min}" max_range="${max}" field_of_view="${ray_fov*M_PI/180}" ray_count="1">
+      <xacro:sonar_sensor name="ray_lfront" parent="${parent_link}" topic="range_lfront" update_rate="${rate}" min_range="${min}" max_range="${max}" field_of_view="${ray_fov*M_PI/180}" ray_count="1">
         <origin xyz="${offX_front} ${offY_left} ${offZ_horizon1}" rpy="0 0 ${45*M_PI/180}" />
       </xacro:sonar_sensor>
       <!-- right -->
-      <xacro:sonar_sensor name="ray_right" parent="${parent_link}" ros_topic="range_right" update_rate="${rate}" min_range="${min}" max_range="${max}" field_of_view="${ray_fov*M_PI/180}" ray_count="1">
+      <xacro:sonar_sensor name="ray_right" parent="${parent_link}" topic="range_right" update_rate="${rate}" min_range="${min}" max_range="${max}" field_of_view="${ray_fov*M_PI/180}" ray_count="1">
         <origin xyz="0 ${offY_right} ${offZ_horizon2}" rpy="0 0 ${-90*M_PI/180}" />
       </xacro:sonar_sensor>
       <!-- left -->
-      <xacro:sonar_sensor name="ray_left" parent="${parent_link}" ros_topic="range_left" update_rate="${rate}" min_range="${min}" max_range="${max}" field_of_view="${ray_fov*M_PI/180}" ray_count="1">
+      <xacro:sonar_sensor name="ray_left" parent="${parent_link}" topic="range_left" update_rate="${rate}" min_range="${min}" max_range="${max}" field_of_view="${ray_fov*M_PI/180}" ray_count="1">
         <origin xyz="0 ${offY_left} ${offZ_horizon2}" rpy="0 0 ${90*M_PI/180}" />
       </xacro:sonar_sensor>
       <!-- right rear -->
-      <xacro:sonar_sensor name="ray_rrear" parent="${parent_link}" ros_topic="range_rrear" update_rate="${rate}" min_range="${min}" max_range="${max}" field_of_view="${ray_fov*M_PI/180}" ray_count="1">
+      <xacro:sonar_sensor name="ray_rrear" parent="${parent_link}" topic="range_rrear" update_rate="${rate}" min_range="${min}" max_range="${max}" field_of_view="${ray_fov*M_PI/180}" ray_count="1">
         <origin xyz="${offX_back} ${offY_right} ${offZ_horizon1}" rpy="0 0 ${-135*M_PI/180}" />
       </xacro:sonar_sensor>
       <!-- left rear -->
-      <xacro:sonar_sensor name="ray_lrear" parent="${parent_link}" ros_topic="range_lrear" update_rate="${rate}" min_range="${min}" max_range="${max}" field_of_view="${ray_fov*M_PI/180}" ray_count="1">
+      <xacro:sonar_sensor name="ray_lrear" parent="${parent_link}" topic="range_lrear" update_rate="${rate}" min_range="${min}" max_range="${max}" field_of_view="${ray_fov*M_PI/180}" ray_count="1">
         <origin xyz="${offX_back} ${offY_left} ${offZ_horizon1}" rpy="0 0 ${135*M_PI/180}" />
       </xacro:sonar_sensor>
       <!-- rear -->
-      <xacro:sonar_sensor name="ray_rear" parent="${parent_link}" ros_topic="range_rear" update_rate="${rate}" min_range="${min}" max_range="${max}" field_of_view="${ray_fov*M_PI/180}" ray_count="1">
+      <xacro:sonar_sensor name="ray_rear" parent="${parent_link}" topic="range_rear" update_rate="${rate}" min_range="${min}" max_range="${max}" field_of_view="${ray_fov*M_PI/180}" ray_count="1">
         <origin xyz="${offX_back} 0 ${offZ_horizon1}" rpy="0 0 ${-180*M_PI/180}" />
       </xacro:sonar_sensor>
       <!-- upward -->
-      <xacro:sonar_sensor name="ray_up" parent="${parent_link}" ros_topic="range_up" update_rate="${rate}" min_range="${min}" max_range="${max}" field_of_view="${ray_fov*M_PI/180}" ray_count="1">
+      <xacro:sonar_sensor name="ray_up" parent="${parent_link}" topic="range_up" update_rate="${rate}" min_range="${min}" max_range="${max}" field_of_view="${ray_fov*M_PI/180}" ray_count="1">
         <origin xyz="0 0 ${offZ_up}" rpy="0 ${-90*M_PI/180} 0" />
       </xacro:sonar_sensor>
       <!-- up front -->
-      <xacro:sonar_sensor name="ray_ufront" parent="${parent_link}" ros_topic="range_ufront" update_rate="${rate}" min_range="${min}" max_range="${max}" field_of_view="${ray_fov*M_PI/180}" ray_count="1">
+      <xacro:sonar_sensor name="ray_ufront" parent="${parent_link}" topic="range_ufront" update_rate="${rate}" min_range="${min}" max_range="${max}" field_of_view="${ray_fov*M_PI/180}" ray_count="1">
         <origin xyz="${offX_front/3} 0 ${offZ_up}" rpy="0 ${-45*M_PI/180} 0" />
       </xacro:sonar_sensor>
       <!-- up rear -->
-      <xacro:sonar_sensor name="ray_urear" parent="${parent_link}" ros_topic="range_urear" update_rate="${rate}" min_range="${min}" max_range="${max}" field_of_view="${ray_fov*M_PI/180}" ray_count="1">
+      <xacro:sonar_sensor name="ray_urear" parent="${parent_link}" topic="range_urear" update_rate="${rate}" min_range="${min}" max_range="${max}" field_of_view="${ray_fov*M_PI/180}" ray_count="1">
         <origin xyz="${offX_back/3} 0 ${offZ_up}" rpy="0 ${-45*M_PI/180} ${180*M_PI/180}" />
       </xacro:sonar_sensor>
       <!-- downward -->
-      <xacro:sonar_sensor name="ray_down" parent="${parent_link}" ros_topic="range_down" update_rate="${rate}" min_range="${min}" max_range="${max}" field_of_view="${ray_fov*M_PI/180}" ray_count="1">
+      <xacro:sonar_sensor name="ray_down" parent="${parent_link}" topic="range_down" update_rate="${rate}" min_range="${min}" max_range="${max}" field_of_view="${ray_fov*M_PI/180}" ray_count="1">
         <origin xyz="0 0 ${offZ_down}" rpy="0 ${90*M_PI/180} 0" />
       </xacro:sonar_sensor>
       <!-- down front -->
-      <xacro:sonar_sensor name="ray_dfront" parent="${parent_link}" ros_topic="range_dfront" update_rate="${rate}" min_range="${min}" max_range="${max}" field_of_view="${ray_fov*M_PI/180}" ray_count="1">
+      <xacro:sonar_sensor name="ray_dfront" parent="${parent_link}" topic="range_dfront" update_rate="${rate}" min_range="${min}" max_range="${max}" field_of_view="${ray_fov*M_PI/180}" ray_count="1">
         <origin xyz="${offX_front/3} 0 ${offZ_down}" rpy="0 ${45*M_PI/180} 0" />
       </xacro:sonar_sensor>
       <!-- down rear -->
-      <xacro:sonar_sensor name="ray_drear" parent="${parent_link}" ros_topic="range_drear" update_rate="${rate}" min_range="${min}" max_range="${max}" field_of_view="${ray_fov*M_PI/180}" ray_count="1">
+      <xacro:sonar_sensor name="ray_drear" parent="${parent_link}" topic="range_drear" update_rate="${rate}" min_range="${min}" max_range="${max}" field_of_view="${ray_fov*M_PI/180}" ray_count="1">
         <origin xyz="${offX_back/3} 0 ${offZ_down}" rpy="0 ${45*M_PI/180} ${180*M_PI/180}" />
       </xacro:sonar_sensor>
